File: KiCAD/guitar-tuner/guitar-tuner.kicad_pcb (KiCad board)
At the start: 2 copper layers, 79.5 x 66 mm, 29 parts, among them J1 Jack-DC, J2 Screw_Terminal_01x04, J3 Screw_Terminal_01x04, SW1 SW_Push, SW2 SW_Push, SW3 SW_Push, SW4 SW_Push, U1 MCP6002-xMC

Commit message: Board_v2
Parts:
- added R4: 0, Resistor_SMD:R_1206_3216Metric, B.Cu at (186.0, 75.0)
- added R5: 0, Resistor_SMD:R_2010_5025Metric, B.Cu at (202.0, 81.5)
- added R6: 0, Resistor_SMD:R_1206_3216Metric, B.Cu at (202.2, 87.8)
- added R7: 0, Resistor_SMD:R_2010_5025Metric, B.Cu at (214.0, 64.5)
- moved J2 30.8 mm to (201.9, 101.5), turned to 0 degrees
- moved C6 13.6 mm to (230.0, 89.0), turned to -90 degrees
- moved C4 10.9 mm to (202.0, 64.0), turned to 0 degrees
- moved R2 6.67 mm to (200.0, 59.0)
- moved RV4 5.21 mm to (192.5, 55.4), turned to 180 degrees
- moved C3 4.92 mm to (201.0, 52.8), turned to -90 degrees
- moved R1 4.20 mm to (225.4, 67.1)
- moved C2 4.20 mm to (225.4, 61.6)
- moved MK1 4.20 mm to (229.0, 62.4)
- moved A2 3.65 mm to (206.3, 92.5)
- moved RV1 2.50 mm to (217.4, 54.9)
- moved H4 1.41 mm to (231.0, 97.0)
- moved C1 1.21 mm to (208.0, 59.8)
- moved C5 1.21 mm to (202.6, 60.4)
- moved RV2 0.50 mm to (217.5, 74.0)
Connections:
- C1 pad 2: +5V -> 5V
- C5 pad 2: +5V -> 5V
- R1 pad 1: +5V -> 5V
- RV4 pad 3: +5V -> 5V
- U1 pad 8: +5V -> 5V
Routing:
- net 5V: track 63.3 -> 127.7 mm, vias 1 -> 0
- net GND: track 227.4 -> 289.5 mm
- net +5V: track 57.5 -> 0.00 mm, vias 2 -> 0
- net Net-(U1A--): track 33.9 -> 48.2 mm, vias 1 -> 0
- net Net-(U1B--): track 36.2 -> 25.0 mm, vias 1 -> 0
- net Net-(A2-1B): track 22.7 -> 13.2 mm
- net Net-(A2-1A): track 19.1 -> 13.2 mm
- net STEP: track 23.2 -> 28.4 mm
- net OUT: track 19.6 -> 23.8 mm
- net 12V: track 63.5 -> 67.4 mm
- net Net-(U1A-+): track 11.8 -> 15.7 mm
- net Net-(A2-2A): track 15.5 -> 13.2 mm
- net Net-(C2-Pad2): track 10.5 -> 8.28 mm
- net Net-(C3-Pad2): track 4.95 -> 3.21 mm
- net DIR: track 26.1 -> 27.7 mm, vias 1 -> 0
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