File: KiCAD/guitar-tuner/guitar-tuner.kicad_sch (KiCad schematic)
At the start: 22 parts, among them J1 Jack-DC, J2 Screw_Terminal_01x04, U1 MCP6002-xMC

Commit message: Board_v1
Parts:
- added D1: LED, LED_THT:LED_D5.0mm, symbol Device:LED
- added J3: Screw_Terminal_01x04, TerminalBlock:TerminalBlock_Xinya_XY308-2.54-4P_1x04_P2.54mm_Horizontal, symbol Connector:Screw_Terminal_01x04
- added R3: 1k, Resistor_SMD:R_0805_2012Metric, symbol Device:R
- added SW1, SW2, SW3: SW_Push, Button_Switch_THT:SW_PUSH_6mm, symbol Switch:SW_Push
- added SW4: SW_Push, Button_Switch_THT:SW_Push_2P2T_Toggle_CK_PVA2xxH1xxxxxxV2, symbol Switch:SW_Push
- C1, C3: footprint Capacitor_THT:C_Radial_D4.0mm_H7.0mm_P1.50mm -> Capacitor_THT:CP_Radial_D5.0mm_P2.50mm
- U1: footprint Package_DFN_QFN:DFN-8-1EP_3x2mm_P0.5mm_EP1.75x1.45mm -> Package_DIP:DIP-8_W7.62mm
Connections:
- net +5V: now also C1.2, C5.2
- net 12V: now also D1.2 (A), SW4.2; no longer J1.1
- net 5V: now also J3.2 (Pin_2)
- net GND: now also C1.1, C5.1, J3.1 (Pin_1), R3.1, SW1.1, SW2.1, SW3.1
- net SW2: now reaches A1.10 (D7)
- net SW2: now also SW2.2
- net SW3: now reaches A1.11 (D8)
- net SW3: now also SW3.2
- net SDA: now reaches A1.23 (A4)
- net SDA: now also J3.3 (Pin_3)
- net SCL: now reaches A1.24 (A5)
- net SCL: now also J3.4 (Pin_4)
- net SW1: now reaches A1.9 (D6)
- net SW1: now also SW1.2
- new net: J1.1, SW4.1
- new net: D1.1 (K), R3.2

Commit message: Board_v2
Parts:
- added R4, R6: 0, Resistor_SMD:R_1206_3216Metric, symbol Device:R
- added R5, R7: 0, Resistor_SMD:R_2010_5025Metric, symbol Device:R
Connections:
- net +5V is gone; now on net 5V: C1.2, C5.2, R1.1, RV4.3, U1.8 (V+)
